File: hardware/heltecv3.kicad_sch (KiCad schematic)
At the start: 0 parts

Commit message: Prel. pin assignments for base station
Other:
- note added: "GPIO33"
- note added: "GPIO34"
- note added: "RX, GPIO44"
- note added: "TX, GPIO43"
Changed lines of the file:
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@@
 	(text "https://resource.heltec.cn/download/WiFi_LoRa_32_V3/HTIT-WB32LA_V3.2.pdf"
 		(exclude_from_sim no)
-		(at 87.63 29.21 0)
+		(at 116.84 26.67 0)
+		(effects
+			(font
+				(size 1.27 1.27)
+			)
+		)
+	)
+	(text "GPIO34"
+		(exclude_from_sim no)
+		(at 156.21 64.77 0)
+		(effects
+			(font
+				(size 1.27 1.27)
+			)
+		)
+	)
+	(text "GPIO33"
+		(exclude_from_sim no)
+		(at 156.21 62.23 0)
+		(effects
+			(font
+				(size 1.27 1.27)
+			)
+		)
+	)
+	(text "RX, GPIO44"
+		(exclude_from_sim no)
+		(at 163.83 77.47 0)
+		(effects
+			(font
+				(size 1.27 1.27)
+			)
+		)
+	)
+	(text "TX, GPIO43"
+		(exclude_from_sim no)
+		(at 163.83 74.93 0)
 		(effects
 			(font
@@
 	)
 	(image
-		(at 76.2 58.42)
+		(at 132.08 63.5)
+		(scale 1.88846)
 		(data "iVBORw0KGgoAAAANSUhEUgAAAwgAAAHBCAIAAABCHwsVAAAAA3NCSVQICAjb4U/gAAAgAElEQVR4"
 			"nOzdeXhU550v+N/7nq1O7SqpSqV9XwAhhAAhwOzGK96NjWPHWdrpSTKddvdtP/dJz53nds/TdyaZ"
@@
 		)
 	)
+	(hierarchical_label "UART_TX"
+		(shape output)
+		(at 146.05 74.93 0)
+		(effects
+			(font
+				(size 1.27 1.27)
+			)
+			(justify left)
+		)
+	)
+	(hierarchical_label "SCL"
+		(shape output)
+		(at 146.05 62.23 0)
+		(effects
+			(font
+				(size 1.27 1.27)
+			)
+			(justify left)
+		)
+	)
 	(hierarchical_label "3V3"
 		(shape output)
-		(at 30.48 25.4 270)
+		(at 76.2 80.01 180)
 		(effects
 			(font
@@
 		)
 	)
-	(hierarchical_label "GND"
+	(hierarchical_label "5V"
+		(shape input)
+		(at 146.05 82.55 0)
+		(effects
+			(font
+				(size 1.27 1.27)
+			)
+			(justify left)
+		)
+	)
+	(hierarchical_label "UART_RX"
 		(shape input)
-		(at 24.13 25.4 90)
+		(at 146.05 77.47 0)
 		(effects
 			(font
@@
 		)
 	)
+	(hierarchical_label "SDA"
+		(shape bidirectional)
+		(at 146.05 64.77 0)
+		(effects
+			(font
+				(size 1.27 1.27)
+			)
+			(justify left)
+		)
+	)
+	(hierarchical_label "GND"
+		(shape input)
+		(at 76.2 85.09 180)
+		(effects
+			(font
+				(size 1.27 1.27)
+			)
+			(justify right)
+		)
+	)
 	(symbol
 		(lib_id "power:GND")
-		(at 24.13 25.4 0)
+		(at 76.2 85.09 90)
 		(unit 1)
 		(exclude_from_sim no)
@@
 		(fields_autoplaced yes)
 		(property "Reference" "#PWR01"
-			(at 24.13 31.75 0)
+			(at 82.55 85.09 0)
 			(effects
 				(font
@@
 		)
 		(property "Value" "GND"
-			(at 24.13 30.48 0)
+			(at 81.28 85.09 0)
 			(effects
 				(font
@@
 		)
 		(property "Footprint" ""
-			(at 24.13 25.4 0)
+			(at 76.2 85.09 0)
 			(effects
 				(font
@@
 		)
 		(property "Datasheet" ""
-			(at 24.13 25.4 0)
+			(at 76.2 85.09 0)
 			(effects
 				(font
@@
 		)
 		(property "Description" "Power symbol creates a global label with name \"GND\" , ground"
-			(at 24.13 25.4 0)
+			(at 76.2 85.09 0)
 			(effects
 				(font
@@
 	)
 	(symbol
+		(lib_id "power:+5V")
+		(at 146.05 82.55 90)
+		(unit 1)
+		(exclude_from_sim no)
+		(in_bom yes)
+		(on_board yes)
+		(dnp no)
+		(fields_autoplaced yes)
+		(property "Reference" "#PWR04"
+			(at 149.86 82.55 0)
+			(effects
+				(font
+					(size 1.27 1.27)
+				)
+				(hide yes)
+			)
+		)
+		(property "Value" "+5V"
+			(at 142.24 82.5499 90)
+			(effects
+				(font
+					(size 1.27 1.27)
+				)
+				(justify left)
+			)
+		)
+		(property "Footprint" ""
+			(at 146.05 82.55 0)
+			(effects
+				(font
+					(size 1.27 1.27)
+				)
+				(hide yes)
+			)
+		)
+		(property "Datasheet" ""
+			(at 146.05 82.55 0)
+			(effects
+				(font
+					(size 1.27 1.27)
+				)
+				(hide yes)
+			)
+		)
+		(property "Description" "Power symbol creates a global label with name \"+5V\""
+			(at 146.05 82.55 0)
+			(effects
+				(font
+					(size 1.27 1.27)
+				)
+				(hide yes)
+			)
+		)
+		(pin "1"
+		)
+		(instances
+			(project ""
+				(path "/586b9940-aa00-4ed6-8067-85ee77ecee7e/f439d00f-b960-4936-bac8-f9fdfbbabd6e"
+					(reference "#PWR04")
+					(unit 1)
+				)
+			)
+		)
+	)
+	(symbol
 		(lib_id "power:+3V3")
-		(at 30.48 25.4 0)
+		(at 76.2 80.01 270)
 		(unit 1)
 		(exclude_from_sim no)
@@
 		(fields_autoplaced yes)
 		(property "Reference" "#PWR02"
-			(at 30.48 29.21 0)
+			(at 72.39 80.01 0)
 			(effects
 				(font
@@
 		)
 		(property "Value" "+3V3"
-			(at 30.48 20.32 0)
+			(at 81.28 80.01 0)
 			(effects
 				(font
@@
 		)
 		(property "Footprint" ""
-			(at 30.48 25.4 0)
+			(at 76.2 80.01 0)
 			(effects
 				(font
@@
 		)
 		(property "Datasheet" ""
-			(at 30.48 25.4 0)
+			(at 76.2 80.01 0)
 			(effects
 				(font
@@
 		)
 		(property "Description" "Power symbol creates a global label with name \"+3V3\""
-			(at 30.48 25.4 0)
+			(at 76.2 80.01 0)
 			(effects
 				(font
