File: hardware/rev2/esp32.kicad_sch (KiCad schematic)
At the start: 47 parts, among them J6 uFL, SW1 SW_Push, SW2 SW_Push, U2 ESP32-S3FN8, Y1 ECS-2520SMV-400-FN-TR

Commit message: changed some components that were on backorder
Parts:
- C15: Mouser Part Number 81-GCM188R72A103KA7D -> 81-GCM188R71H103KA7J
- J6: Mouser Part Number 712-CONMHF1-SMD-G-T -> 712-CONUFL001-SMD-T
- R36, R37: Mouser Part Number (none) -> 71-CRCW06034K70JNEBC
Changed lines of the file:
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@@
 			)
 		)
-		(property "Datasheet" "https://www.te.com/commerce/DocumentDelivery/DDEController?Action=srchrtrv&DocNm=conmhf1-smd-g-t-ds&DocType=Data+Sheet&DocLang=English&DocFormat=pdf&PartCntxt=CONMHF1-SMD-G-T"
+		(property "Datasheet" "https://www.te.com/commerce/DocumentDelivery/DDEController?Action=srchrtrv&DocNm=CONUFL001-SMD-T&DocType=Data+Sheet&DocLang=English&DocFormat=pdf&PartCntxt=CONUFL001-SMD-T"
 			(at 257.81 151.13 0)
 			(hide yes)
@@
 			)
 		)
-		(property "Mouser Part Number" "712-CONMHF1-SMD-G-T "
+		(property "Mouser Part Number" "712-CONUFL001-SMD-T "
 			(at 257.81 151.13 90)
 			(hide yes)
@@
 			)
 		)
-		(property "Datasheet" ""
+		(property "Datasheet" "https://www.vishay.com/docs/20035/dcrcwe3.pdf"
 			(at 24.13 135.89 0)
 			(hide yes)
@@
 			)
 		)
-		(property "Mouser Part Number" ""
+		(property "Mouser Part Number" "71-CRCW06034K70JNEBC"
 			(at 24.13 135.89 90)
 			(hide yes)
@@
 			)
 		)
-		(property "Datasheet" ""
+		(property "Datasheet" "https://www.vishay.com/docs/20035/dcrcwe3.pdf"
 			(at 24.13 146.05 0)
 			(hide yes)
@@
 			)
 		)
-		(property "Mouser Part Number" ""
+		(property "Mouser Part Number" "71-CRCW06034K70JNEBC"
 			(at 24.13 146.05 90)
 			(hide yes)
@@
 			)
 		)
-		(property "Datasheet" "https://pim.murata.com/asset/pim4/ceramicCapacitorSMD/GCM188R72A103KA37-01C-EN_PDF_CERAMICCAPACITORSMD"
+		(property "Datasheet" "https://pim.murata.com/asset/pim4/ceramicCapacitorSMD/GCM188R71H103KA37-01C-EN_PDF_CERAMICCAPACITORSMD"
 			(at 44.45 80.01 0)
 			(hide yes)
@@
 			)
 		)
-		(property "Mouser Part Number" "81-GCM188R72A103KA7D"
+		(property "Mouser Part Number" "81-GCM188R71H103KA7J"
 			(at 44.45 80.01 0)
 			(hide yes)
