File: hardware/rev2/sx1262.kicad_sch (KiCad schematic)
At the start: 40 parts, among them Q1 SS8050, U3 SX1262IMLTRT, U4 PE4259, Y2 TXO-20CSMV-320

Commit message: no clue, don't remember
Other:
- moved on the sheet: R24
Changed lines of the file:
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@@
 	(title_block
 		(title "LoRa Based Cat Tracker")
-		(date "2026-04-28")
+		(date "2026-03-31")
 		(rev "2.0.1")
 		(company "Group 10")
@@
 	(rectangle
 		(start 29.845 92.075)
-		(end 83.82 187.325)
+		(end 86.36 187.325)
 		(stroke
 			(width 0)
@@
 	(rectangle
 		(start 210.82 40.005)
-		(end 243.84 69.85)
+		(end 250.19 69.85)
 		(stroke
 			(width 0)
@@
 	)
 	(junction
+		(at 82.55 114.3)
+		(diameter 0)
+		(color 0 0 0 0)
+	)
+	(junction
 		(at 55.88 85.09)
 		(diameter 0)
@@
 	)
 	(junction
-		(at 80.01 114.3)
-		(diameter 0)
-		(color 0 0 0 0)
-	)
-	(junction
 		(at 170.18 83.82)
 		(diameter 0)
@@
 	(wire
 		(pts
-			(xy 80.01 139.7) (xy 80.01 114.3)
+			(xy 82.55 139.7) (xy 82.55 114.3)
 		)
 		(stroke
@@
 	(wire
 		(pts
-			(xy 72.39 114.3) (xy 80.01 114.3)
+			(xy 72.39 114.3) (xy 82.55 114.3)
 		)
 		(stroke
@@
 	(wire
 		(pts
-			(xy 80.01 139.7) (xy 63.5 139.7)
+			(xy 82.55 139.7) (xy 63.5 139.7)
 		)
 		(stroke
@@
 	(symbol
 		(lib_id "Device:R")
-		(at 80.01 110.49 0)
+		(at 82.55 110.49 0)
 		(mirror y)
 		(unit 1)
@@
 		(dnp no)
 		(property "Reference" "R24"
-			(at 77.47 109.2199 0)
+			(at 80.01 109.2199 0)
 			(show_name no)
 			(do_not_autoplace no)
@@
 		)
 		(property "Value" "10 k"
-			(at 77.47 111.7599 0)
+			(at 80.01 111.7599 0)
 			(show_name no)
 			(do_not_autoplace no)
@@
 		)
 		(property "Footprint" "Resistor_SMD:R_0603_1608Metric_Pad0.98x0.95mm_HandSolder"
-			(at 81.788 110.49 90)
+			(at 84.328 110.49 90)
 			(hide yes)
 			(show_name no)
@@
 		)
 		(property "Datasheet" "https://www.vishay.com/docs/20035/dcrcwe3.pdf"
-			(at 80.01 110.49 0)
+			(at 82.55 110.49 0)
 			(hide yes)
 			(show_name no)
@@
 		)
 		(property "Description" "Resistor"
-			(at 80.01 110.49 0)
+			(at 82.55 110.49 0)
 			(hide yes)
 			(show_name no)
@@
 		)
 		(property "KLC_S3.3" ""
-			(at 80.01 110.49 90)
+			(at 82.55 110.49 90)
 			(hide yes)
 			(show_name no)
@@
 		)
 		(property "KLC_S4.1" ""
-			(at 80.01 110.49 90)
+			(at 82.55 110.49 90)
 			(hide yes)
 			(show_name no)
@@
 		)
 		(property "Sim.Type" ""
-			(at 80.01 110.49 0)
+			(at 82.55 110.49 0)
 			(hide yes)
 			(show_name no)
@@
 		)
 		(property "Mouser Part Number" "71-CRCW060310K0JNEAC"
-			(at 80.01 110.49 0)
+			(at 82.55 110.49 0)
 			(hide yes)
 			(show_name no)
@@
 		)
 		(property "KLC_S5.1" ""
-			(at 80.01 110.49 0)
+			(at 82.55 110.49 0)
 			(hide yes)
 			(show_name no)
@@
 	(symbol
 		(lib_id "power:+3V3")
-		(at 80.01 106.68 0)
+		(at 82.55 106.68 0)
 		(unit 1)
 		(body_style 1)
@@
 		(fields_autoplaced yes)
 		(property "Reference" "#PWR068"
-			(at 80.01 110.49 0)
+			(at 82.55 110.49 0)
 			(hide yes)
 			(show_name no)
@@
 		)
 		(property "Value" "+3V3"
-			(at 80.01 101.6 0)
+			(at 82.55 101.6 0)
 			(show_name no)
 			(do_not_autoplace no)
@@
 		)
 		(property "Footprint" ""
-			(at 80.01 106.68 0)
+			(at 82.55 106.68 0)
 			(hide yes)
 			(show_name no)
@@
 		)
 		(property "Datasheet" ""
-			(at 80.01 106.68 0)
+			(at 82.55 106.68 0)
 			(hide yes)
 			(show_name no)
@@
 		)
 		(property "Description" "Power symbol creates a global label with name \"+3V3\""
-			(at 80.01 106.68 0)
+			(at 82.55 106.68 0)
 			(hide yes)
 			(show_name no)
@@
 		(in_pos_files yes)
 		(dnp no)
-		(fields_autoplaced yes)
 		(property "Reference" "L15"
-			(at 194.31 62.23 90)
+			(at 194.31 60.96 90)
 			(show_name no)
 			(do_not_autoplace no)
@@
 		)
 		(property "Value" "17 nH"
-			(at 194.31 64.77 90)
+			(at 194.31 63.5 90)
 			(show_name no)
 			(do_not_autoplace no)
@@
 		(in_pos_files yes)
 		(dnp no)
-		(fields_autoplaced yes)
 		(property "Reference" "C43"
 			(at 76.2 116.8399 0)
@@
 		)
 		(property "Value" "1000 pF"
-			(at 76.2 119.3799 0)
+			(at 73.66 120.65 0)
 			(show_name no)
 			(do_not_autoplace no)
